File: FC_PCB/FC_PCB.kicad_sch (KiCad schematic)
At the start: 4 parts

Commit message: Commit final hard
Other:
- sheet ESP_MCU ports: added none; removed ESP_SPI2_CS0, ESP_SPI2_MISO, ESP_SPI2_MOSI, ESP_SPI2_SCK, ESP_UART2_RX, ESP_UART2_TX
- sheet ESP_PERIPHE ports: added none; removed CONN_I2C_SCL, CONN_I2C_SDA, CONN_SPI_CLK, CONN_SPI_CS, CONN_SPI_MISO, CONN_SPI_MOSI, CONN_UART_RX, CONN_UART_TX
- company: (none) -> Aliou LY
- title: (none) -> FC-GAOL
