File: FC_PCB/espMCU.kicad_sch (KiCad schematic)
At the start: 26 parts, among them J3 USB_C_Receptacle_USB2.0_16P, Q1 EMH3, SW1 RESET, SW2 RESET, U1 ESP32-S3-MINI-1, U2 CP2102N-Axx-xQFN24

Commit message: Commit final hard
Connections:
- net ESP_UART2_TX is gone; now on net ESP_I2C_SDA: U1.10 (GPIO6/TOUCH6/ADC1_CH5)
- net ESC_PWM3: no longer U1.35 (MTCK/GPIO39/CLK_OUT3/SUBSPICS1)
- net ESP_HOLD: now also U1.30 (GPIO48/SPICLK_N/SUBSPICLK_N_DIFF); no longer U1.26 (GPIO26)
- net ESP_I2C_SCL: now also U1.8 (GPIO4/TOUCH4/ADC1_CH3); no longer U1.9 (GPIO5/TOUCH5/ADC1_CH4)
- net ESP_I2C_SDA: no longer U1.8 (GPIO4/TOUCH4/ADC1_CH3)
- net ESP_SPI3_CS0: now also U1.33 (SPIDQS/GPIO37/FSPIQ/SUBSPIQ); no longer U1.29 (SPIIO5/GPIO34/FSPICS0/SUBSPICS0)
- net ESP_SPI3_MISO: now also U1.32 (SPIIO7/GPIO36/FSPICLK/SUBSPICLK); no longer U1.33 (SPIDQS/GPIO37/FSPIQ/SUBSPIQ)
- net ESP_SPI3_MOSI: now also U1.28 (SPIIO4/GPIO33/FSPIHD/SUBSPIHD); no longer U1.31 (SPIIO6/GPIO35/FSPID/SUBSPID)
- net ESP_SPI3_SCK: now also U1.29 (SPIIO5/GPIO34/FSPICS0/SUBSPICS0); no longer U1.32 (SPIIO7/GPIO36/FSPICLK/SUBSPICLK)
- net ESP_WP: now also U1.31 (SPIIO6/GPIO35/FSPID/SUBSPID); no longer U1.28 (SPIIO4/GPIO33/FSPIHD/SUBSPIHD)
- net GPIO_8: now also U1.9 (GPIO5/TOUCH5/ADC1_CH4); no longer U1.12 (GPIO8/TOUCH8/ADC1_CH7/SUBSPICS1)
- net ESP_SPI2_CS0: no longer names the net of U1.14 (GPIO10/TOUCH10/ADC1_CH9/FSPICS0/FSPIIO4/SUBSPICS0)
- net ESP_SPI2_MISO: no longer names the net of U1.17 (GPIO13/TOUCH13/ADC2_CH2/FSPIQ/FSPIIO7/SUBSPIQ)
- net ESP_SPI2_MOSI: no longer names the net of U1.15 (GPIO11/TOUCH11/ADC2_CH0/FSPID/FSPIIO5/SUBSPID)
- net ESP_SPI2_SCK: no longer names the net of U1.16 (GPIO12/TOUCH12/ADC2_CH1/FSPICLK/FSPIIO6/SUBSPICLK)
- net ESP_UART2_RX: no longer names the net of U1.11 (GPIO7/TOUCH7/ADC1_CH6)
- new net ESC_PWM4: U1.35 (MTCK/GPIO39/CLK_OUT3/SUBSPICS1)
- no-connect marks 20 -> 26
Changed lines of the file:
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@@
+	)
+	(no_connect
+		(at 125.73 139.7)
 	)
 	(no_connect
@@
 	)
 	(no_connect
+		(at 125.73 142.24)
+	)
+	(no_connect
 		(at 34.29 114.3)
 	)
@@
 	)
 	(no_connect
+		(at 125.73 149.86)
+	)
+	(no_connect
 		(at 125.73 167.64)
 	)
@@
 	)
 	(no_connect
+		(at 125.73 154.94)
+	)
+	(no_connect
 		(at 261.62 67.31)
 	)
@@
 	)
 	(no_connect
+		(at 125.73 147.32)
+	)
+	(no_connect
 		(at 261.62 39.37)
 	)
@@
 	)
 	(no_connect
-		(at 125.73 177.8)
+		(at 125.73 152.4)
+	)
+	(no_connect
+		(at 34.29 165.1)
 	)
 	(no_connect
@@
 		)
 	)
-	(hierarchical_label "ESP_I2C_SDA"
-		(shape input)
-		(at 125.73 132.08 0)
-		(effects
-			(font
-				(size 1.27 1.27)
-				(thickness 0.1588)
-			)
-			(justify left)
-		)
-	)
-	(hierarchical_label "GPIO_9"
-		(shape input)
-		(at 125.73 144.78 0)
+	(hierarchical_label "ESP_SPI3_SCK"
+		(shape input)
+		(at 34.29 170.18 180)
 		(effects
 			(font
@@
 				(bold yes)
 			)
-			(justify left)
-		)
-	)
-	(hierarchical_label "GPIO_8"
-		(shape input)
-		(at 125.73 142.24 0)
+			(justify right)
+		)
+	)
+	(hierarchical_label "GPIO_9"
+		(shape input)
+		(at 125.73 144.78 0)
 		(effects
 			(font
@@
 		)
 	)
-	(hierarchical_label "ESP_SPI2_SCK"
-		(shape input)
-		(at 125.73 152.4 0)
+	(hierarchical_label "ESP_UART1_RX"
+		(shape input)
+		(at 125.73 162.56 0)
+		(effects
+			(font
+				(size 1.27 1.27)
+				(thickness 0.1588)
+			)
+			(justify left)
+		)
+	)
+	(hierarchical_label "ESP_SPI3_MISO"
+		(shape input)
+		(at 34.29 175.26 180)
 		(effects
 			(font
@@
 				(bold yes)
 			)
-			(justify left)
+			(justify right)
 		)
 	)
 	(hierarchical_label "ESP_HOLD"
 		(shape input)
-		(at 34.29 165.1 180)
+		(at 125.73 177.8 0)
 		(effects
 			(font
@@
 				(bold yes)
 			)
-			(justify right)
-		)
-	)
-	(hierarchical_label "ESP_UART1_RX"
-		(shape input)
-		(at 125.73 162.56 0)
-		(effects
-			(font
-				(size 1.27 1.27)
-				(thickness 0.1588)
-			)
 			(justify left)
 		)
 	)
-	(hierarchical_label "ESP_UART2_RX"
-		(shape input)
-		(at 125.73 139.7 0)
-		(effects
-			(font
-				(size 1.27 1.27)
-				(thickness 0.1588)
-			)
-			(justify left)
-		)
-	)
-	(hierarchical_label "ESP_SPI3_MOSI"
+	(hierarchical_label "ESP_WP"
 		(shape input)
 		(at 34.29 172.72 180)
@@
 		)
 	)
-	(hierarchical_label "ESP_UART2_TX"
-		(shape input)
-		(at 125.73 137.16 0)
-		(effects
-			(font
-				(size 1.27 1.27)
-				(thickness 0.1588)
-			)
-			(justify left)
-		)
-	)
-	(hierarchical_label "ESP_SPI3_CS0"
-		(shape input)
-		(at 34.29 170.18 180)
+	(hierarchical_label "GPIO_21"
+		(shape input)
+		(at 125.73 165.1 0)
 		(effects
 			(font
@@
 				(bold yes)
 			)
+			(justify left)
+		)
+	)
+	(hierarchical_label "ESP_UART1_TX"
+		(shape input)
+		(at 125.73 160.02 0)
+		(effects
+			(font
+				(size 1.27 1.27)
+				(thickness 0.1588)
+			)
+			(justify left)
+		)
+	)
+	(hierarchical_label "ESP_I2C_SDA"
+		(shape input)
+		(at 125.73 137.16 0)
+		(effects
+			(font
+				(size 1.27 1.27)
+				(thickness 0.1588)
+			)
+			(justify left)
+		)
+	)
+	(hierarchical_label "ESC_PWM3"
+		(shape input)
+		(at 34.29 121.92 180)
+		(effects
+			(font
+				(size 1.27 1.27)
+			)
 			(justify right)
 		)
 	)
-	(hierarchical_label "GPIO_21"
-		(shape input)
-		(at 125.73 165.1 0)
+	(hierarchical_label "ESC_PWM4"
+		(shape input)
+		(at 34.29 119.38 180)
+		(effects
+			(font
+				(size 1.27 1.27)
+			)
+			(justify right)
+		)
+	)
+	(hierarchical_label "ESP_SPI3_MOSI"
+		(shape input)
+		(at 34.29 167.64 180)
 		(effects
 			(font
@@
 				(bold yes)
 			)
-			(justify left)
-		)
-	)
-	(hierarchical_label "ESP_SPI2_MISO"
-		(shape input)
-		(at 125.73 154.94 0)
+			(justify right)
+		)
+	)
+	(hierarchical_label "ESP_SPI3_CS0"
+		(shape input)
+		(at 34.29 177.8 180)
 		(effects
 			(font
@@
 				(bold yes)
 			)
-			(justify left)
-		)
-	)
-	(hierarchical_label "ESP_UART1_TX"
-		(shape input)
-		(at 125.73 160.02 0)
-		(effects
-			(font
-				(size 1.27 1.27)
-				(thickness 0.1588)
-			)
-			(justify left)
-		)
-	)
-	(hierarchical_label "ESC_PWM3"
-		(shape input)
-		(at 34.29 121.92 180)
-		(effects
-			(font
-				(size 1.27 1.27)
-			)
 			(justify right)
 		)
 	)
-	(hierarchical_label "ESC_PWM3"
-		(shape input)
-		(at 34.29 119.38 180)
-		(effects
-			(font
-				(size 1.27 1.27)
-			)
-			(justify right)
-		)
-	)
-	(hierarchical_label "ESP_SPI2_MOSI"
-		(shape input)
-		(at 125.73 149.86 0)
+	(hierarchical_label "GPIO_8"
+		(shape input)
+		(at 125.73 134.62 0)
 		(effects
 			(font
@@
 		)
 	)
-	(hierarchical_label "ESP_SPI3_MISO"
-		(shape input)
-		(at 34.29 177.8 180)
+	(hierarchical_label "ESP_I2C_SCL"
+		(shape input)
+		(at 125.73 132.08 0)
+		(effects
+			(font
+				(size 1.27 1.27)
+				(thickness 0.1588)
+			)
+			(justify left)
+		)
+	)
+	(hierarchical_label "GPIO_14"
+		(shape input)
+		(at 125.73 157.48 0)
 		(effects
 			(font
@@
 				(bold yes)
 			)
+			(justify left)
+		)
+	)
+	(hierarchical_label "ESC_PWM1"
+		(shape input)
+		(at 34.29 127 180)
+		(effects
+			(font
+				(size 1.27 1.27)
+			)
 			(justify right)
-		)
-	)
-	(hierarchical_label "ESP_SPI3_SCK"
-		(shape input)
-		(at 34.29 175.26 180)
-		(effects
-			(font
-				(size 1.27 1.27)
-				(thickness 0.254)
-				(bold yes)
-			)
-			(justify right)
-		)
-	)
-	(hierarchical_label "ESP_SPI2_CS0"
-		(shape input)
-		(at 125.73 147.32 0)
-		(effects
-			(font
-				(size 1.27 1.27)
-				(thickness 0.254)
-				(bold yes)
-			)
-			(justify left)
-		)
-	)
-	(hierarchical_label "GPIO_14"
-		(shape input)
-		(at 125.73 157.48 0)
-		(effects
-			(font
-				(size 1.27 1.27)
-				(thickness 0.254)
-				(bold yes)
-			)
-			(justify left)
-		)
-	)
-	(hierarchical_label "ESP_I2C_SCL"
-		(shape input)
-		(at 125.73 134.62 0)
-		(effects
-			(font
-				(size 1.27 1.27)
-				(thickness 0.1588)
-			)
-			(justify left)
-		)
-	)
-	(hierarchical_label "ESC_PWM1"
-		(shape input)
-		(at 34.29 127 180)
-		(effects
-			(font
-				(size 1.27 1.27)
-			)
-			(justify right)
-		)
-	)
-	(hierarchical_label "ESP_WP"
-		(shape input)
-		(at 34.29 167.64 180)
-		(effects
-			(font
-				(size 1.27 1.27)
-				(thickness 0.254)
-				(bold yes)
-			)
-			(justify right)
